Commit message: created robot_descriptor parameter and dummy link to the urdf

File: src/startup/urdf/robot.urdf (robot description, URDF)
Before this commit: robot MARS-2026-robot, 5 links, 4 joints
Links:
- added link dummy_root
Joints:
- added joint dummy_root_joint: type fixed, parent dummy_root, child base_link, origin xyz=0 0 0 rpy=0 0 0
