Commit message: use ros2-control for mujoco

File: src/startup/urdf/robot/urdf/mujoco_actuators.urdf.xacro (robot description, xacro)
@@ -13,5 +13,5 @@
     <!-- Calculate position feedback gain (kp) -->
     <xacro:property name="kp" value="${effort}" />
-    <!-- Create position actuator -->
+    <!-- Create velocity actuator -->
     <velocity
       name="vel_actuator_${joint}"

File: src/startup/urdf/robot/urdf/robot.urdf (robot description, URDF)
Before this commit: robot robot, 11 links, 10 joints
Links:
- link frame_assembly: mass 30 -> 40
Joints:
- joint front_left_drum_joint: limit effort=10 velocity=10 -> effort=1000 velocity=10
- joint front_left_wheel_joint: limit effort=10 velocity=10 -> effort=1000 velocity=10
- joint front_right_wheel_joint: limit effort=10 velocity=10 -> effort=1000 velocity=10
- joint rear_left_wheel_joint: limit effort=10 velocity=10 -> effort=1000 velocity=10
- joint rear_right_wheel_joint: limit effort=10 velocity=10 -> effort=1000 velocity=10

File: src/startup/urdf/robot/urdf/robot.urdf.xacro (robot description, xacro)
@@ -25,36 +25,51 @@
   <xacro:include filename="$(find startup)/urdf/robot/urdf/robot.urdf" />
   <xacro:include filename="$(find startup)/urdf/robot/urdf/ros2_control.urdf.xacro" />
-  <xacro:robot_ros2_control use_sim="$(arg use_sim)" mujoco_effort="$(arg mujoco_effort)" />
-  <xacro:if value="$(arg use_sim)">
-      <mujoco>
-          <compiler meshdir="$(arg mujoco_model_path)/meshes"
-                    discardvisual="false"
-                    autolimits="$(arg autolimits)"
-                    balanceinertia="$(arg balanceinertia)"
-          />
-          <option integrator="$(arg integrator)"
-                  gravity="$(arg gravity)"
-                  impratio="$(arg impratio)"
-                  cone="$(arg cone)"
-                  solver="$(arg solver)"
-                  noslip_iterations="$(arg noslip_iterations)">
-              <flag multiccd="$(arg multiccd)" />
-          </option>
-          <!-- Create actuators to use position control -->
-          <xacro:unless value="$(arg mujoco_effort)">
-              <xacro:include filename="$(find startup)/urdf/robot/urdf/mujoco_actuators.urdf.xacro" />
-              <xacro:create_mujoco_actuators/>
-          </xacro:unless>
-          <contact>
-            <pair geom1="front_arm_collision_0" geom2="frame_assembly_collision_0" friction="1 0.005 0.0001" solimp="0.99 0.99 0.001"/>
-            <pair geom1="rear_arm_collision_0" geom2="frame_assembly_collision_1" friction="1 0.005 0.0001" solimp="0.99 0.99 0.001"/>
-          </contact>
-          <!-- <body name="front_arm" gravcomp="1" />
-          <body name="rear_arm" gravcomp="1" />
-          <body name="front_left_drum" gravcomp="1" />
-          <body name="front_right_drum" gravcomp="1" />
-          <body name="rear_left_drum" gravcomp="1" />
-          <body name="rear_right_drum" gravcomp="1" /> -->
-      </mujoco>
-  </xacro:if>
+  <mujoco_inputs>
+    <raw_inputs>
+        <!-- <compiler meshdir="$(arg mujoco_model_path)/meshes"
+                  discardvisual="false"
+                  autolimits="$(arg autolimits)"
+                  balanceinertia="$(arg balanceinertia)"
+        />
+        <option integrator="$(arg integrator)"
+                gravity="$(arg gravity)"
+                impratio="$(arg impratio)"
+                cone="$(arg cone)"
+                solver="$(arg solver)"
+                noslip_iterations="$(arg noslip_iterations)">
+            <flag multiccd="$(arg multiccd)" />
+        </option> -->
+        <option integrator="implicitfast"/>
+        <default>
+          <default class="visual">
+            <geom group="2" type="mesh" contype="0" conaffinity="0"/>
+          </default>
+          <default class="collision">
+            <geom group="3" type="mesh"/>
+          </default>
+        </default>
+        <!-- Create actuators to use position control -->
+        <xacro:include filename="$(find startup)/urdf/robot/urdf/mujoco_actuators.urdf.xacro" />
+        <xacro:create_mujoco_actuators/>
+        <contact>
+          <!-- <pair geom1="front_arm_collision_mesh0" geom2="frame_assembly_collision_mesh0" friction="1 0.005 0.0001" solimp="0.99 0.99 0.001"/>
+          <pair geom1="rear_arm_collision_mesh0" geom2="frame_assembly_collision_mesh1" friction="1 0.005 0.0001" solimp="0.99 0.99 0.001"/> -->
+        </contact>
+    </raw_inputs>
+    <processed_inputs>
+      <!-- <modify_element type="body" name="front_arm" gravcomp="1" />
+      <modify_element type="body" name="rear_arm" gravcomp="1" /> -->
+      <!-- <modify_element type="joint" name="front_arm_joint" armature="125.0" />
+      <modify_element type="joint" name="rear_arm_joint" armature="125.0" />
+      <modify_element type="joint" name="front_left_drum_joint" armature="125.0" />
+      <modify_element type="joint" name="front_right_drum_joint" armature="125.0" />
+      <modify_element type="joint" name="rear_left_drum_joint" armature="125.0" />
+      <modify_element type="joint" name="rear_right_drum_joint" armature="125.0" />
+      <modify_element type="joint" name="front_left_wheel_joint" armature="125.0" />
+      <modify_element type="joint" name="front_right_wheel_joint" armature="125.0" />
+      <modify_element type="joint" name="rear_left_wheel_joint" armature="125.0" />
+      <modify_element type="joint" name="rear_right_wheel_joint" armature="125.0" /> -->
+    </processed_inputs>
+  </mujoco_inputs>
+  <xacro:robot_ros2_control use_sim="$(arg use_sim)" mujoco_effort="$(arg mujoco_effort)" mujoco_model_path="$(arg mujoco_model_path)" />
 </robot>

File: src/startup/urdf/robot/urdf/ros2_control.urdf.xacro (robot description, xacro)
@@ -2,9 +2,12 @@
 <robot xmlns:xacro="http://www.ros.org/wiki/xacro">
 <xacro:macro name="robot_ros2_control"
-             params="use_sim mujoco_effort">
-  <ros2_control name="RobotHardwareSystem" type="system">
+             params="use_sim mujoco_effort mujoco_model_path">
+  <ros2_control name="MujocoSystem" type="system">
     <hardware>
       <xacro:if value="$(arg use_sim)">
-        <plugin>mujoco_ros2_control/MujocoSystem</plugin>
+        <plugin>mujoco_ros2_control/MujocoSystemInterface</plugin>
+        <param name="headless">false</param>
+        <!-- <param name="mujoco_model">${mujoco_model_path}</param> -->
+        <param name="sim_speed_factor">1.0</param>
       </xacro:if>
       <xacro:unless value="$(arg use_sim)">

Commit message: re-refactor arms to use JointGroupVelocityController

File: src/startup/urdf/robot/urdf/mujoco_actuators.urdf.xacro (robot description, xacro)
@@ -59,8 +59,6 @@
       <xacro:create_mujoco_velocity_actuator joint_limits="${joint_limits}" joint="front_arm_joint" />
       <xacro:create_mujoco_velocity_actuator joint_limits="${joint_limits}" joint="rear_arm_joint" />
-      <xacro:create_mujoco_velocity_actuator joint_limits="${joint_limits}" joint="front_left_drum_joint" />
-      <xacro:create_mujoco_velocity_actuator joint_limits="${joint_limits}" joint="front_right_drum_joint" />
-      <xacro:create_mujoco_velocity_actuator joint_limits="${joint_limits}" joint="rear_left_drum_joint" />
-      <xacro:create_mujoco_velocity_actuator joint_limits="${joint_limits}" joint="rear_right_drum_joint" />
+      <xacro:create_mujoco_velocity_actuator joint_limits="${joint_limits}" joint="front_drum_joint" />
+      <xacro:create_mujoco_velocity_actuator joint_limits="${joint_limits}" joint="rear_drum_joint" />
     </actuator>
   </xacro:macro>

File: src/startup/urdf/robot/urdf/robot.urdf (robot description, URDF)
Before this commit: robot robot, 19 links, 18 joints
Joints:
- removed joint front_left_drum_joint
- removed joint rear_left_drum_joint
- added joint front_drum_joint: type continuous, parent front_arm, child drum, origin xyz=0.357187 0.0476885 0.0381 rpy=1.51327e-16 -1.41588e-16 -1.5708, axis 0 0 1, limit effort=1000 velocity=10
- added joint rear_drum_joint: type continuous, parent rear_arm, child rear_left_drum, origin xyz=0.357188 0.0476885 -0.0381 rpy=6.51149e-31 -1.66571e-30 -8.18079e-17, axis 0 0 1, limit effort=10 velocity=10
- joint front_right_drum_joint: mimic (none) -> joint=front_drum_joint multiplier=1 offset=0
- joint rear_right_drum_joint: mimic (none) -> joint=rear_drum_joint multiplier=1 offset=0

File: src/startup/urdf/robot/urdf/ros2_control.urdf.xacro (robot description, xacro)
@@ -39,8 +39,6 @@
     <xacro:configure_joint joint_name="front_arm_joint" initial_position="0.0" />
     <xacro:configure_joint joint_name="rear_arm_joint" initial_position="0.0" />
-    <xacro:configure_joint joint_name="front_left_drum_joint" initial_position="0.0" />
-    <xacro:configure_joint joint_name="front_right_drum_joint" initial_position="0.0" />
-    <xacro:configure_joint joint_name="rear_left_drum_joint" initial_position="0.0" />
-    <xacro:configure_joint joint_name="rear_right_drum_joint" initial_position="0.0" />
+    <xacro:configure_joint joint_name="front_drum_joint" initial_position="0.0" />
+    <xacro:configure_joint joint_name="rear_drum_joint" initial_position="0.0" />
     <sensor name="front_camera">
       <param name="frame_name">front_camera_color_mujoco_frame</param>
