Commit message: added second depth camera, and renamed a bunch of stuff to make more sense

File: src/startup/urdf/robot/urdf/rgbd.gazebo.xacro (robot description, xacro)
@@ -2,6 +2,6 @@
 <robot xmlns:xacro="http://wiki.ros.org/xacro">
   <!-- Functional RGB-D approximation, not a model of RealSense stereo/IMU. -->
-  <xacro:macro name="d435i_rgbd" params="parent">
-    <link name="d435i_link">
+  <xacro:macro name="rgbd_camera" params="parent name xyz yaw">
+    <link name="${name}_link">
       <inertial>
         <mass value="0.075"/>
@@ -10,26 +10,25 @@
       <visual>
         <geometry><box size="0.025 0.09 0.025"/></geometry>
-        <material name="d435i_material"><color rgba="0.2 0.2 0.2 1"/></material>
+        <material name="rgbd_material"><color rgba="0.2 0.2 0.2 1"/></material>
       </visual>
     </link>
-    <joint name="d435i_mount_joint" type="fixed">
+    <joint name="${name}_mount_joint" type="fixed">
       <parent link="${parent}"/>
-      <child link="d435i_link"/>
-      <!-- Blue side is the physical front (-Y in frame_assembly).
-           Mount above the legacy rear_camera position; tilt down 15 degrees. -->
-      <origin xyz="0.1159 -0.2921 0.1308" rpy="0 ${pi / 12} ${-pi / 2}"/>
+      <child link="${name}_link"/>
+      <!-- Mount on either side of the chassis; tilt down 15 degrees. -->
+      <origin xyz="${xyz}" rpy="0 ${pi / 12} ${yaw}"/>
     </joint>
-    <link name="d435i_optical_frame"/>
-    <joint name="d435i_optical_joint" type="fixed">
-      <parent link="d435i_link"/>
-      <child link="d435i_optical_frame"/>
+    <link name="${name}_optical_frame"/>
+    <joint name="${name}_optical_joint" type="fixed">
+      <parent link="${name}_link"/>
+      <child link="${name}_optical_frame"/>
       <origin xyz="0 0 0" rpy="${-pi / 2} 0 ${-pi / 2}"/>
     </joint>
-    <gazebo reference="d435i_link">
-      <sensor name="d435i_rgbd" type="rgbd_camera">
+    <gazebo reference="${name}_link">
+      <sensor name="${name}_rgbd" type="rgbd_camera">
         <always_on>true</always_on>
         <update_rate>30</update_rate>
-        <topic>/d435i</topic>
-        <gz_frame_id>d435i_optical_frame</gz_frame_id>
+        <topic>/${name}</topic>
+        <gz_frame_id>${name}_optical_frame</gz_frame_id>
         <camera>
           <!-- Shared RGB/depth geometry; these are simulation defaults. -->
@@ -44,5 +43,5 @@
             <clip><near>0.1</near><far>10.0</far></clip>
           </depth_camera>
-          <camera_info_topic>/d435i/camera_info</camera_info_topic>
+          <camera_info_topic>/${name}/camera_info</camera_info_topic>
         </camera>
       </sensor>

File: src/startup/urdf/robot/urdf/robot.urdf.xacro (robot description, xacro)
@@ -1,7 +1,7 @@
 <?xml version="1.0" ?>
 <robot xmlns:xacro="http://wiki.ros.org/xacro" name="robot">
-  <xacro:arg name="enable_d435i" default="false"/>
+  <xacro:arg name="enable_rgbd" default="false"/>
   <xacro:arg name="enable_lidar" default="false"/>
-  <xacro:include filename="$(find startup)/urdf/robot/urdf/d435i.gazebo.xacro" />
+  <xacro:include filename="$(find startup)/urdf/robot/urdf/rgbd.gazebo.xacro" />
   <xacro:include filename="$(find startup)/urdf/robot/urdf/robot.urdf" />
   <xacro:include filename="$(find startup)/urdf/robot/urdf/ros2_control.urdf.xacro" />
@@ -36,7 +36,10 @@
   <xacro:gazebo_camera name="front"/>
   <xacro:gazebo_camera name="rear"/>
-  <xacro:if value="$(arg enable_d435i)">
+  <xacro:if value="$(arg enable_rgbd)">
     <xacro:if value="${'$(arg robot_backend)' == 'gazebo'}">
-      <xacro:d435i_rgbd parent="frame_assembly"/>
+      <xacro:rgbd_camera parent="frame_assembly" name="rgbd_blue"
+                        xyz="0.1159 -0.2921 0.1308" yaw="${-pi / 2}"/>
+      <xacro:rgbd_camera parent="frame_assembly" name="rgbd_orange"
+                        xyz="0.1159 0.2921 0.1308" yaw="${pi / 2}"/>
     </xacro:if>
   </xacro:if>
