Commit message: attempted making navigation not chud (it is still lowk chud)

File: src/startup/urdf/robot/urdf/robot.urdf.xacro (robot description, xacro)
@@ -5,4 +5,13 @@
   <xacro:include filename="$(find startup)/urdf/robot/urdf/rgbd.gazebo.xacro" />
   <xacro:include filename="$(find startup)/urdf/robot/urdf/robot.urdf" />
+  <!-- Navigation convention: +X points toward the blue drums (-Y of CAD).
+       Keep the CAD frame and UI drive reversal unchanged. A selectable-front
+       implementation can add a separate logical frame/command adapter later. -->
+  <link name="base_link" />
+  <joint name="blue_forward_base_joint" type="fixed">
+    <parent link="base_link" />
+    <child link="frame_assembly" />
+    <origin xyz="0 0 0" rpy="0 0 ${pi / 2}" />
+  </joint>
   <xacro:include filename="$(find startup)/urdf/robot/urdf/ros2_control.urdf.xacro" />
   <xacro:robot_ros2_control robot_backend="$(arg robot_backend)" />

Commit message: add (untested) robot serial hardware

File: src/startup/urdf/robot/urdf/robot.urdf.xacro (robot description, xacro)
@@ -15,5 +15,5 @@
   </joint>
   <xacro:include filename="$(find startup)/urdf/robot/urdf/ros2_control.urdf.xacro" />
-  <xacro:robot_ros2_control robot_backend="$(arg robot_backend)" />
+  <xacro:robot_ros2_control robot_backend="$(arg robot_backend)" serial_port="$(arg serial_port)" />
   <xacro:macro name="gazebo_camera" params="name">
     <gazebo reference="${name}_camera_link">

File: src/startup/urdf/robot/urdf/ros2_control.urdf.xacro (robot description, xacro)
@@ -1,5 +1,5 @@
 <?xml version="1.0"?>
 <robot xmlns:xacro="http://www.ros.org/wiki/xacro">
-<xacro:macro name="robot_ros2_control" params="robot_backend">
+<xacro:macro name="robot_ros2_control" params="robot_backend serial_port">
   <ros2_control name="RobotSystem" type="system">
     <hardware>
@@ -11,5 +11,7 @@
       </xacro:if>
       <xacro:if value="${robot_backend == 'serial'}">
-        <plugin>mock_components/GenericSystem</plugin>
+        <plugin>robot_serial_hardware/RobotSerialHardware</plugin>
+        <param name="port">${serial_port}</param>
+        <param name="baudrate">115200</param>
       </xacro:if>
     </hardware>
