Commit message: add rviz and cameras to simulation. add gstreamer to simulation launch file

File: src/startup/urdf/robot/urdf/robot.urdf (robot description, URDF)
Before this commit: robot robot, 11 links, 10 joints
Links:
- added link front_camera_color_frame
- added link front_camera_color_mujoco_frame
- added link front_camera_color_optical_frame
- added link front_camera_link, mass 1; collision box size=0.05 0.05 0.05; visual box size=0.05 0.05 0.05
- added link rear_camera_color_frame
- added link rear_camera_color_mujoco_frame
- added link rear_camera_color_optical_frame
- added link rear_camera_link, mass 1; collision box size=0.05 0.05 0.05; visual box size=0.05 0.05 0.05
Joints:
- added joint front_camera_color_frame_joint: type fixed, parent front_camera_link, child front_camera_color_frame, origin xyz=0 0 0 rpy=0 0 0
- added joint front_camera_color_mujoco_joint: type fixed, parent front_camera_color_optical_frame, child front_camera_color_mujoco_frame, origin xyz=0 0 0 rpy=3.14159 0 0
- added joint front_camera_color_optical_frame_joint: type fixed, parent front_camera_color_frame, child front_camera_color_optical_frame, origin xyz=0 0 0 rpy=-1.5708 -1.5708 0
- added joint front_camera_joint: type fixed, parent frame_assembly, child front_camera_link, origin xyz=-0.1159 0.2921 0.0508 rpy=-1.5708 1.0472 -1.5708
- added joint rear_camera_color_frame_joint: type fixed, parent rear_camera_link, child rear_camera_color_frame, origin xyz=0 0 0 rpy=0 0 0
- added joint rear_camera_color_mujoco_joint: type fixed, parent rear_camera_color_optical_frame, child rear_camera_color_mujoco_frame, origin xyz=0 0 0 rpy=3.14159 0 0
- added joint rear_camera_color_optical_frame_joint: type fixed, parent rear_camera_color_frame, child rear_camera_color_optical_frame, origin xyz=0 0 0 rpy=-1.5708 -1.5708 0
- added joint rear_camera_joint: type fixed, parent frame_assembly, child rear_camera_link, origin xyz=0.1159 -0.2921 0.0508 rpy=-1.5708 1.0472 1.5708

File: src/startup/urdf/robot/urdf/robot.urdf.xacro (robot description, xacro)
@@ -18,8 +18,9 @@
   <xacro:arg name="mujoco_effort" default="false" /> <!-- position actuators must be defined before using them -->
   <link name="world"/>
-  <joint name="world_joint" type="floating">
+  <joint name="base_link" type="floating">
+    <axis xyz="0 0 0" rpy="0 0 0"/>
+    <origin xyz="0 0 0.5" rpy="0 0 0"/>
     <parent link="world"/>
     <child link="frame_assembly"/>
-    <origin xyz="0 0 0.0" rpy="0 0 2.00"/>
   </joint>
   <xacro:include filename="$(find startup)/urdf/robot/urdf/robot.urdf" />
@@ -70,4 +71,6 @@
       <modify_element type="joint" name="rear_left_wheel_joint" armature="125.0" />
       <modify_element type="joint" name="rear_right_wheel_joint" armature="125.0" /> -->
+      <camera site="front_camera_color_optical_frame" name="front_camera" mode="fixed" fovy="58" resolution="640 480"/>
+      <camera site="rear_camera_color_optical_frame" name="rear_camera" mode="fixed" fovy="58" resolution="640 480"/>
     </processed_inputs>
   </mujoco_inputs>

File: src/startup/urdf/robot/urdf/ros2_control.urdf.xacro (robot description, xacro)
@@ -43,4 +43,16 @@
     <xacro:configure_joint joint_name="rear_left_drum_joint" initial_position="0.0" />
     <xacro:configure_joint joint_name="rear_right_drum_joint" initial_position="0.0" />
+    <sensor name="front_camera">
+      <param name="frame_name">front_camera_color_mujoco_frame</param>
+      <param name="info_topic">/front_camera/color/camera_info</param>
+      <param name="image_topic">/front_camera/image_raw</param>
+      <param name="depth_topic">/front_camera/depth/image_raw</param>
+    </sensor>
+    <sensor name="rear_camera">
+      <param name="frame_name">rear_camera_color_mujoco_frame</param>
+      <param name="info_topic">/rear_camera/color/camera_info</param>
+      <param name="image_topic">/rear_camera/image_raw</param>
+      <param name="depth_topic">/rear_camera/depth/image_raw</param>
+    </sensor>
   </ros2_control>
 </xacro:macro>

Commit message: refactor gazebo startup to be in startup package; modify deploy.sh to use launch arguments

File: src/startup/urdf/robot/urdf/robot.urdf (robot description, URDF)
Before this commit: robot robot, 19 links, 18 joints
Links:
- removed link front_camera_color_mujoco_frame
- removed link rear_camera_color_mujoco_frame
- link drum: mass 1 -> 1.5
- link frame_assembly: mass 40 -> 30
- link front_left_wheel: mass 1.7 -> 1.1
- link front_right_drum: mass 1 -> 1.5
- link front_right_wheel: mass 1.7 -> 1.1
- link rear_left_drum: mass 1 -> 1.5
- link rear_left_wheel: mass 1.7 -> 1.1
- link rear_right_drum: mass 1 -> 1.5
- link rear_right_wheel: mass 1.7 -> 1.1
Joints:
- removed joint front_camera_color_mujoco_joint
- removed joint rear_camera_color_mujoco_joint
- joint front_arm_joint: limit effort=1000 velocity=1000 -> lower=-1.2 upper=0.2 effort=1000 velocity=2.0; type continuous -> revolute
- joint front_camera_joint: origin xyz=-0.1159 0.2921 0.0508 rpy=-1.5708 1.0472 -1.5708 -> xyz=-0.1159 0.2921 0.0508 rpy=-1.5708 1.308996939 -1.5708
- joint front_right_drum_joint: axis 0 0 1 -> (none); limit effort=10 velocity=10 -> (none); mimic joint=front_drum_joint multiplier=1 offset=0 -> (none); origin xyz=0.357187 0.0476885 -0.0381 rpy=-7.85046e-17 4.12558e-32 -3.14159 -> xyz=0 0 -0.0762 rpy=0 0 -1.57079; parent front_arm -> drum; type continuous -> fixed
- joint rear_arm_joint: limit effort=1000 velocity=1000 -> lower=-1.2 upper=0.2 effort=1000 velocity=2.0; type continuous -> revolute
- joint rear_camera_joint: origin xyz=0.1159 -0.2921 0.0508 rpy=-1.5708 1.0472 1.5708 -> xyz=0.1159 -0.2921 0.0508 rpy=-1.5708 1.308996939 1.5708
- joint rear_drum_joint: limit effort=10 velocity=10 -> effort=1000 velocity=10
- joint rear_right_drum_joint: axis 0 0 1 -> (none); limit effort=10 velocity=10 -> (none); mimic joint=rear_drum_joint multiplier=1 offset=0 -> (none); origin xyz=0.357187 0.0476885 0.0381 rpy=3.90337e-31 5.47109e-32 -3.14159 -> xyz=-0.000001 0 0.0762 rpy=0 0 -3.14159; parent rear_arm -> rear_left_drum; type continuous -> fixed

File: src/startup/urdf/robot/urdf/robot.urdf.xacro (robot description, xacro)
@@ -1,78 +1,47 @@
 <?xml version="1.0" ?>
-<robot xmlns:xacro="http://wiki.ros.org/xacro" name="$(arg name)">
-  <!-- MuJoCo Config -->
-  <!-- Mujoco compiler options -->
-  <xacro:arg name="mujoco_model_path" default="/tmp/mujoco" />
-  <xacro:arg name="autolimits" default="true" />
-  <xacro:arg name="balanceinertia" default="true" />
-  <!-- Mujoco options -->
-  <xacro:arg name="integrator" default="implicitfast" />
-  <xacro:arg name="gravity" default="0 0 -9.81" />
-  <xacro:arg name="impratio" default="1" />
-  <xacro:arg name="integrator" default="implicitfast" />
-  <xacro:arg name="cone" default="elliptic" />
-  <xacro:arg name="solver" default="Newton" />
-  <xacro:arg name="noslip_iterations" default="3" />
-  <xacro:arg name="multiccd" default="disable" />
-  <xacro:arg name="use_sim" default="true" />
-  <xacro:arg name="mujoco_effort" default="false" /> <!-- position actuators must be defined before using them -->
-  <link name="world"/>
-  <joint name="base_link" type="floating">
-    <axis xyz="0 0 0" rpy="0 0 0"/>
-    <origin xyz="0 0 0.5" rpy="0 0 0"/>
-    <parent link="world"/>
-    <child link="frame_assembly"/>
-  </joint>
+<robot xmlns:xacro="http://wiki.ros.org/xacro" name="robot">
   <xacro:include filename="$(find startup)/urdf/robot/urdf/robot.urdf" />
   <xacro:include filename="$(find startup)/urdf/robot/urdf/ros2_control.urdf.xacro" />
-  <mujoco_inputs>
-    <raw_inputs>
-        <!-- <compiler meshdir="$(arg mujoco_model_path)/meshes"
-                  discardvisual="false"
-                  autolimits="$(arg autolimits)"
-                  balanceinertia="$(arg balanceinertia)"
-        />
-        <option integrator="$(arg integrator)"
-                gravity="$(arg gravity)"
-                impratio="$(arg impratio)"
-                cone="$(arg cone)"
-                solver="$(arg solver)"
-                noslip_iterations="$(arg noslip_iterations)">
-            <flag multiccd="$(arg multiccd)" />
-        </option> -->
-        <option integrator="implicitfast"/>
-        <default>
-          <default class="visual">
-            <geom group="2" type="mesh" contype="0" conaffinity="0"/>
-          </default>
-          <default class="collision">
-            <geom group="3" type="mesh"/>
-          </default>
-        </default>
-        <!-- Create actuators to use position control -->
-        <xacro:include filename="$(find startup)/urdf/robot/urdf/mujoco_actuators.urdf.xacro" />
-        <xacro:create_mujoco_actuators/>
-        <contact>
-          <!-- <pair geom1="front_arm_collision_mesh0" geom2="frame_assembly_collision_mesh0" friction="1 0.005 0.0001" solimp="0.99 0.99 0.001"/>
-          <pair geom1="rear_arm_collision_mesh0" geom2="frame_assembly_collision_mesh1" friction="1 0.005 0.0001" solimp="0.99 0.99 0.001"/> -->
-        </contact>
-    </raw_inputs>
-    <processed_inputs>
-      <!-- <modify_element type="body" name="front_arm" gravcomp="1" />
-      <modify_element type="body" name="rear_arm" gravcomp="1" /> -->
-      <!-- <modify_element type="joint" name="front_arm_joint" armature="125.0" />
-      <modify_element type="joint" name="rear_arm_joint" armature="125.0" />
-      <modify_element type="joint" name="front_left_drum_joint" armature="125.0" />
-      <modify_element type="joint" name="front_right_drum_joint" armature="125.0" />
-      <modify_element type="joint" name="rear_left_drum_joint" armature="125.0" />
-      <modify_element type="joint" name="rear_right_drum_joint" armature="125.0" />
-      <modify_element type="joint" name="front_left_wheel_joint" armature="125.0" />
-      <modify_element type="joint" name="front_right_wheel_joint" armature="125.0" />
-      <modify_element type="joint" name="rear_left_wheel_joint" armature="125.0" />
-      <modify_element type="joint" name="rear_right_wheel_joint" armature="125.0" /> -->
-      <camera site="front_camera_color_optical_frame" name="front_camera" mode="fixed" fovy="58" resolution="640 480"/>
-      <camera site="rear_camera_color_optical_frame" name="rear_camera" mode="fixed" fovy="58" resolution="640 480"/>
-    </processed_inputs>
-  </mujoco_inputs>
-  <xacro:robot_ros2_control use_sim="$(arg use_sim)" mujoco_effort="$(arg mujoco_effort)" mujoco_model_path="$(arg mujoco_model_path)" />
+  <xacro:robot_ros2_control robot_backend="$(arg robot_backend)" />
+  <xacro:macro name="gazebo_camera" params="name">
+    <gazebo reference="${name}_camera_link">
+      <sensor name="${name}_camera" type="camera">
+        <!-- Map Gazebo +X forward / +Z up to optical +Z forward / -Y up.
+             The optical joint uses RPY (-pi/2, -pi/2, 0); yaw alone
+             aligns the viewing direction but leaves the image rolled 90 degrees. -->
+        <pose>0 0 0 ${-pi / 2} 0 ${pi / 2}</pose>
+        <always_on>true</always_on>
+        <update_rate>$(arg camera_update_rate)</update_rate>
+        <topic>/${name}_camera/image_raw</topic>
+        <gz_frame_id>${name}_camera_color_optical_frame</gz_frame_id>
+        <camera>
+          <!-- MuJoCo uses a 58 degree vertical FOV at a 4:3 aspect ratio. -->
+          <horizontal_fov>${2 * atan(tan(58 * pi / 360) * 4 / 3)}</horizontal_fov>
+          <image>
+            <width>640</width>
+            <height>480</height>
+            <format>R8G8B8</format>
+          </image>
+          <clip>
+            <near>0.05</near>
+            <far>100</far>
+          </clip>
+        </camera>
+      </sensor>
+    </gazebo>
+  </xacro:macro>
+  <xacro:gazebo_camera name="front"/>
+  <xacro:gazebo_camera name="rear"/>
+  <!-- ============================= -->
+  <!-- Gazebo ros2_control plugin    -->
+  <!-- ============================= -->
+  <gazebo>
+    <plugin
+        filename="libgz_ros2_control-system.so"
+        name="gz_ros2_control::GazeboSimROS2ControlPlugin">
+      <parameters>
+        $(find startup)/config/controllers.yaml
+      </parameters>
+    </plugin>
+  </gazebo>
 </robot>

File: src/startup/urdf/robot/urdf/ros2_control.urdf.xacro (robot description, xacro)
@@ -1,56 +1,33 @@
 <?xml version="1.0"?>
 <robot xmlns:xacro="http://www.ros.org/wiki/xacro">
-<xacro:macro name="robot_ros2_control"
-             params="use_sim mujoco_effort mujoco_model_path">
-  <ros2_control name="MujocoSystem" type="system">
+<xacro:macro name="robot_ros2_control" params="robot_backend">
+  <ros2_control name="RobotSystem" type="system">
     <hardware>
-      <xacro:if value="$(arg use_sim)">
-        <plugin>mujoco_ros2_control/MujocoSystemInterface</plugin>
-        <param name="headless">false</param>
-        <!-- <param name="mujoco_model">${mujoco_model_path}</param> -->
-        <param name="sim_speed_factor">1.0</param>
+      <xacro:if value="${robot_backend == 'gazebo'}">
+        <plugin>gz_ros2_control/GazeboSimSystem</plugin>
       </xacro:if>
-      <xacro:unless value="$(arg use_sim)">
+      <xacro:if value="${robot_backend == 'mock'}">
         <plugin>mock_components/GenericSystem</plugin>
-      </xacro:unless>
+      </xacro:if>
+      <xacro:if value="${robot_backend == 'serial'}">
+        <plugin>mock_components/GenericSystem</plugin>
+      </xacro:if>
     </hardware>
-    <xacro:macro name="configure_joint" params="joint_name initial_position">
+    <xacro:macro name="configure_joint" params="joint_name">
       <joint name="${joint_name}">
-        <xacro:if value="${mujoco_effort}">
-          <command_interface name="effort"/>
-        </xacro:if>
-        <xacro:unless value="${mujoco_effort}">
-          <command_interface name="velocity"/>
-          <command_interface name="position"/>
-        </xacro:unless>
-        <state_interface name="position">
-          <param name="initial_value">${initial_position}</param>
-        </state_interface>
-        <state_interface name="velocity">
-          <param name="initial_value">0.0</param>
-        </state_interface>
+        <command_interface name="velocity"/>
+        <state_interface name="position"/>
+        <state_interface name="velocity"/>
         <state_interface name="effort"/>
       </joint>
     </xacro:macro>
-    <xacro:configure_joint joint_name="front_left_wheel_joint" initial_position="0.0" />
-    <xacro:configure_joint joint_name="front_right_wheel_joint" initial_position="0.0" />
-    <xacro:configure_joint joint_name="rear_left_wheel_joint" initial_position="0.0" />
-    <xacro:configure_joint joint_name="rear_right_wheel_joint" initial_position="0.0" />
-    <xacro:configure_joint joint_name="front_arm_joint" initial_position="0.0" />
-    <xacro:configure_joint joint_name="rear_arm_joint" initial_position="0.0" />
-    <xacro:configure_joint joint_name="front_drum_joint" initial_position="0.0" />
-    <xacro:configure_joint joint_name="rear_drum_joint" initial_position="0.0" />
-    <sensor name="front_camera">
-      <param name="frame_name">front_camera_color_mujoco_frame</param>
-      <param name="info_topic">/front_camera/color/camera_info</param>
-      <param name="image_topic">/front_camera/image_raw</param>
-      <param name="depth_topic">/front_camera/depth/image_raw</param>
-    </sensor>
-    <sensor name="rear_camera">
-      <param name="frame_name">rear_camera_color_mujoco_frame</param>
-      <param name="info_topic">/rear_camera/color/camera_info</param>
-      <param name="image_topic">/rear_camera/image_raw</param>
-      <param name="depth_topic">/rear_camera/depth/image_raw</param>
-    </sensor>
+    <xacro:configure_joint joint_name="front_left_wheel_joint" />
+    <xacro:configure_joint joint_name="front_right_wheel_joint" />
+    <xacro:configure_joint joint_name="rear_left_wheel_joint" />
+    <xacro:configure_joint joint_name="rear_right_wheel_joint" />
+    <xacro:configure_joint joint_name="front_arm_joint" />
+    <xacro:configure_joint joint_name="rear_arm_joint" />
+    <xacro:configure_joint joint_name="front_drum_joint" />
+    <xacro:configure_joint joint_name="rear_drum_joint" />
   </ros2_control>
 </xacro:macro>

Commit message: add lidar simulation to gazebo

File: src/startup/urdf/robot/urdf/robot.urdf (robot description, URDF)
Before this commit: robot robot, 17 links, 16 joints
Links:
- added link unilidar_link, mass 0.5; collision cylinder length=0.08 radius=0.05; visual cylinder length=0.08 radius=0.05
Joints:
- added joint unilidar_joint: type fixed, parent frame_assembly, child unilidar_link, origin xyz=0 0 0.05 rpy=0 0 0

File: src/startup/urdf/robot/urdf/robot.urdf.xacro (robot description, xacro)
@@ -40,4 +40,61 @@
     </xacro:if>
   </xacro:if>
+  <gazebo reference="unilidar_link">
+    <!-- 1. 3D LiDAR Sensor Profile (Unitree L2 Specifications) -->
+    <sensor name="unilidar_cloud" type="gpu_lidar">
+      <pose>0 0 0 0 0 0</pose>
+      <update_rate>10</update_rate>
+      <ray>
+        <scan>
+          <horizontal>
+            <samples>360</samples>
+            <resolution>1</resolution>
+            <min_angle>-3.14159</min_angle>
+            <max_angle>3.14159</max_angle>
+          </horizontal>
+          <vertical>
+            <samples>32</samples> <!-- Unitree L2 features a dense vertical profile -->
+            <resolution>1</resolution>
+            <min_angle>-0.261799</min_angle> <!-- -15 deg -->
+            <max_angle>0.261799</max_angle>  <!-- +15 deg -->
+          </vertical>
+        </scan>
+        <range>
+          <min>0.1</min>
+          <max>30.0</max>
+          <resolution>0.01</resolution>
+        </range>
+      </ray>
+      <always_on>true</always_on>
+      <visualize>false</visualize>
+      <topic>unilidar/cloud</topic>
+      <gz_frame_id>unilidar_link</gz_frame_id>
+    </sensor>
+    <!-- 2. Integrated IMU Sensor Profile (with exact internal offset) -->
+    <sensor name="unilidar_imu" type="imu">
+      <always_on>true</always_on>
+      <update_rate>200</update_rate> <!-- Fast update rate for LIO pipelines -->
+      <visualize>false</visualize>
+      <topic>unilidar/imu</topic>
+      <!-- Accurate physical hardware offset inside Unitree L2 housing -->
+      <pose>-0.007698 -0.014655 0.00667 0 0 0</pose>
+      <gz_frame_id>unilidar_link</gz_frame_id>
+      <imu>
+        <angular_velocity>
+          <x><noise type="gaussian"><mean>0.0</mean><stddev>2e-4</stddev></noise></x>
+          <y><noise type="gaussian"><mean>0.0</mean><stddev>2e-4</stddev></noise></y>
+          <z><noise type="gaussian"><mean>0.0</mean><stddev>2e-4</stddev></noise></z>
+        </angular_velocity>
+        <linear_acceleration>
+          <x><noise type="gaussian"><mean>0.0</mean><stddev>1.7e-2</stddev></noise></x>
+          <y><noise type="gaussian"><mean>0.0</mean><stddev>1.7e-2</stddev></noise></y>
+          <z><noise type="gaussian"><mean>0.0</mean><stddev>1.7e-2</stddev></noise></z>
+        </linear_acceleration>
+      </imu>
+    </sensor>
+  </gazebo>
+  <gazebo reference="unilidar_joint">
+    <disableFixedJointLumping>true</disableFixedJointLumping>
+  </gazebo>
   <!-- ============================= -->
   <!-- Gazebo ros2_control plugin    -->
@@ -51,4 +108,8 @@
       </parameters>
     </plugin>
+    <plugin
+      filename="gz-sim-imu-system"
+      name="gz::sim::systems::Imu">
+    </plugin>
   </gazebo>
 </robot>

File: src/startup/urdf/robot/urdf/ros2_control.urdf.xacro (robot description, xacro)
@@ -30,4 +30,16 @@
     <xacro:configure_joint joint_name="front_drum_joint" />
     <xacro:configure_joint joint_name="rear_drum_joint" />
+    <sensor name="unilidar_imu">
+      <state_interface name="orientation.x"/>
+      <state_interface name="orientation.y"/>
+      <state_interface name="orientation.z"/>
+      <state_interface name="orientation.w"/>
+      <state_interface name="angular_velocity.x"/>
+      <state_interface name="angular_velocity.y"/>
+      <state_interface name="angular_velocity.z"/>
+      <state_interface name="linear_acceleration.x"/>
+      <state_interface name="linear_acceleration.y"/>
+      <state_interface name="linear_acceleration.z"/>
+    </sensor>
   </ros2_control>
 </xacro:macro>

Commit message: fixed collision issues (changed wheels collision to be cylinders), and made the heightmap for craters use a lot less lines.

File: src/startup/urdf/robot/urdf/robot.urdf (robot description, URDF)
Before this commit: robot robot, 18 links, 17 joints
Links:
- link front_left_wheel: geometry collision cylinder length=0.079375 radius=0.1778; visual mesh filename=file://$(find startup)/urdf/robot/assets/wheel.stl
- link front_right_wheel: geometry collision cylinder length=0.079375 radius=0.1778; visual mesh filename=file://$(find startup)/urdf/robot/assets/wheel.stl
- link rear_left_wheel: geometry collision cylinder length=0.079375 radius=0.1778; visual mesh filename=file://$(find startup)/urdf/robot/assets/wheel.stl
- link rear_right_wheel: geometry collision cylinder length=0.079375 radius=0.1778; visual mesh filename=file://$(find startup)/urdf/robot/assets/wheel.stl

Commit message: fixed some directional issues; dump auto should do blue side predominately, and front camera should be defined as on the front of the robot

File: src/startup/urdf/robot/urdf/robot.urdf (robot description, URDF)
Before this commit: robot robot, 18 links, 17 joints
Joints:
- joint front_camera_joint: origin xyz=-0.1159 0.2921 0.0508 rpy=-1.5708 1.308996939 -1.5708 -> xyz=0.1159 -0.2921 0.0508 rpy=-1.5708 1.308996939 1.5708
- joint rear_camera_joint: origin xyz=0.1159 -0.2921 0.0508 rpy=-1.5708 1.308996939 1.5708 -> xyz=-0.1159 0.2921 0.0508 rpy=-1.5708 1.308996939 -1.5708
