Commit message: fixed drums and arms for gazebo

File: src/lunabotics_simulation/urdf/robot/urdf/robot_gazebo.urdf (robot description, URDF)
Before this commit: robot robot, 17 links, 16 joints
Joints:
- removed joint front_left_drum_joint
- removed joint rear_left_drum_joint
- added joint front_drum_joint: type continuous, parent front_arm, child drum, origin xyz=0.357187 0.0476885 0.0381 rpy=1.51327e-16 -1.41588e-16 -1.5708, axis 0 0 1, limit effort=1000 velocity=10
- added joint rear_drum_joint: type continuous, parent rear_arm, child rear_left_drum, origin xyz=0.357188 0.0476885 -0.0381 rpy=6.51149e-31 -1.66571e-30 -8.18079e-17, axis 0 0 1, limit effort=10 velocity=10
- joint front_right_drum_joint: axis 0 0 1 -> (none); limit effort=10 velocity=10 -> (none); origin xyz=0.357187 0.0476885 -0.0381 rpy=-7.85046e-17 4.12558e-32 -3.14159 -> xyz=0 0 -0.0762 rpy=0 0 -1.57079; parent front_arm -> drum; type continuous -> fixed
- joint rear_right_drum_joint: axis 0 0 1 -> (none); limit effort=10 velocity=10 -> (none); origin xyz=0.357187 0.0476885 0.0381 rpy=3.90337e-31 5.47109e-32 -3.14159 -> xyz=-0.000001 0 0.0762 rpy=0 0 -3.14159; parent rear_arm -> rear_left_drum; type continuous -> fixed

File: src/lunabotics_simulation/urdf/robot/urdf/ros2_control_gazebo.urdf.xacro (robot description, xacro)
@@ -45,5 +45,5 @@
       </joint>
       <!-- Drums -->
-      <joint name="front_left_drum_joint">
+      <joint name="front_drum_joint">
         <command_interface name="velocity"/>
         <state_interface name="position"/>
@@ -51,17 +51,5 @@
         <state_interface name="effort"/>
       </joint>
-      <joint name="front_right_drum_joint">
-        <command_interface name="velocity"/>
-        <state_interface name="position"/>
-        <state_interface name="velocity"/>
-        <state_interface name="effort"/>
-      </joint>
-      <joint name="rear_left_drum_joint">
-        <command_interface name="velocity"/>
-        <state_interface name="position"/>
-        <state_interface name="velocity"/>
-        <state_interface name="effort"/>
-      </joint>
-      <joint name="rear_right_drum_joint">
+      <joint name="rear_drum_joint">
         <command_interface name="velocity"/>
         <state_interface name="position"/>

Commit message: made dockerfile set ENV RMW_IMPLMENTATION when built, and added cameras to the gazebo installation. Also added zenoh to gazebo.launch, effectively deprecating setup_terminal.sh

File: src/lunabotics_simulation/urdf/robot/urdf/robot_gazebo.urdf (robot description, URDF)
Before this commit: robot robot, 17 links, 16 joints
Joints:
- joint front_camera_joint: origin xyz=-0.1159 0.2921 0.0508 rpy=-1.5708 1.0472 -1.5708 -> xyz=-0.1159 0.2921 0.0508 rpy=-1.5708 1.308996939 -1.5708
- joint rear_camera_joint: origin xyz=0.1159 -0.2921 0.0508 rpy=-1.5708 1.0472 1.5708 -> xyz=0.1159 -0.2921 0.0508 rpy=-1.5708 1.308996939 1.5708

File: src/lunabotics_simulation/urdf/robot/urdf/robot_gazebo.urdf.xacro (robot description, xacro)
@@ -3,4 +3,5 @@
     xmlns:xacro="http://www.ros.org/wiki/xacro"
     name="robot">
+  <xacro:arg name="camera_update_rate" default="30.0"/>
   <!-- ============================= -->
   <!-- Common robot                  -->
@@ -14,4 +15,33 @@
       filename="$(find lunabotics_simulation)/urdf/robot/urdf/ros2_control_gazebo.urdf.xacro"/>
   <xacro:ros2_control_gazebo/>
+  <xacro:macro name="gazebo_camera" params="name">
+    <gazebo reference="${name}_camera_link">
+      <sensor name="${name}_camera" type="camera">
+        <!-- Map Gazebo +X forward / +Z up to optical +Z forward / -Y up.
+             The optical joint uses RPY (-pi/2, -pi/2, 0); yaw alone
+             aligns the viewing direction but leaves the image rolled 90 degrees. -->
+        <pose>0 0 0 ${-pi / 2} 0 ${pi / 2}</pose>
+        <always_on>true</always_on>
+        <update_rate>$(arg camera_update_rate)</update_rate>
+        <topic>/${name}_camera/image_raw</topic>
+        <gz_frame_id>${name}_camera_color_optical_frame</gz_frame_id>
+        <camera>
+          <!-- MuJoCo uses a 58 degree vertical FOV at a 4:3 aspect ratio. -->
+          <horizontal_fov>${2 * atan(tan(58 * pi / 360) * 4 / 3)}</horizontal_fov>
+          <image>
+            <width>640</width>
+            <height>480</height>
+            <format>R8G8B8</format>
+          </image>
+          <clip>
+            <near>0.05</near>
+            <far>100</far>
+          </clip>
+        </camera>
+      </sensor>
+    </gazebo>
+  </xacro:macro>
+  <xacro:gazebo_camera name="front"/>
+  <xacro:gazebo_camera name="rear"/>
   <!-- ============================= -->
   <!-- Gazebo ros2_control plugin    -->

Commit message: simulation is frfr setup now; all our autonomy from last year works, and I set up some basic physics. i also recolored the drums and wheels for funsies. oh i also fixed a few bugs with teleop n stuff

File: src/lunabotics_simulation/urdf/robot/urdf/robot_gazebo.urdf (robot description, URDF)
Before this commit: robot robot, 17 links, 16 joints
Links:
- link drum: mass 1 -> 1.5
- link frame_assembly: mass 40 -> 30
- link front_left_wheel: mass 1.7 -> 1.1
- link front_right_drum: mass 1 -> 1.5
- link front_right_wheel: mass 1.7 -> 1.1
- link rear_left_drum: mass 1 -> 1.5
- link rear_left_wheel: mass 1.7 -> 1.1
- link rear_right_drum: mass 1 -> 1.5
- link rear_right_wheel: mass 1.7 -> 1.1
Joints:
- joint front_arm_joint: limit effort=1000 velocity=1000 -> lower=-1.2 upper=0.2 effort=1000 velocity=2.0; type continuous -> revolute
- joint rear_arm_joint: limit effort=1000 velocity=1000 -> lower=-1.2 upper=0.2 effort=1000 velocity=2.0; type continuous -> revolute
- joint rear_drum_joint: limit effort=10 velocity=10 -> effort=1000 velocity=10
